Commit message: Upload new version

File: catkin_ws/src/arm_description/urdf/arm.xacro (robot description, xacro)
@@ -3,5 +3,5 @@
 <!-- This document describes the robot model -->
 <!--   Machenical Practice Testing Version   -->
-<!--        Last editted: 11/01, 2018        -->
+<!--        Last editted: 11/18, 2018        -->
 <!--            Editor: Wolf Chen            -->
 <robot name="arm" xmlns:xacro="http://www.ros.org/wiki/xacro">
@@ -11,4 +11,5 @@
   <!-- END - Include -->
   <!-- BGN - Robot Description -->
+  <!-- Body -->
   <arm_cylinder name="${l0b}"
                 mass="${base_mass}"
@@ -18,10 +19,10 @@
                 izz="1"
                 radius="${base_r}" length="${base_l}"/>
-  <arm_joint name="${l0b}_to_${m0b}" type="revolute"
-             axis_xyz="0 0 1"
-             limit_angle="1.57"
-             origin_rpy="0 0 0" origin_xyz="0 0 ${base_l}"
-             parent="${l0b}"
-             child="${m0b}"/>
+  <arm_joint_trans name="${l0b}_to_${m0b}" type="revolute"
+                   axis_xyz="0 0 1"
+                   limit="1.57"
+                   origin_rpy="0 0 0" origin_xyz="0 0 ${base_l}"
+                   parent="${l0b}"
+                   child="${m0b}"/>
   <arm_box name="${m0b}"
            mass="${basem_mass}"
@@ -31,10 +32,10 @@
            izz="1"
            size="${basem_w} ${basem_l} ${basem_h}"/>
-  <arm_joint name="${m0b}_to_${l01}" type="revolute"
-             axis_xyz="0 1 0"
-             limit_angle="1.57"
-             origin_rpy="0 0 0" origin_xyz="0 0 ${basem_h}"
-             parent="${m0b}"
-             child="${l01}"/>
+  <arm_joint_trans name="${m0b}_to_${l01}" type="revolute"
+                   axis_xyz="0 1 0"
+                   limit="1.57"
+                   origin_rpy="0 0 0" origin_xyz="0 0 ${basem_h}"
+                   parent="${m0b}"
+                   child="${l01}"/>
   <arm_box name="${l01}"
            mass="${body_mass}"
@@ -44,9 +45,9 @@
            izz="1"
            size="${body_w} ${body_l} ${body_h}"/>
-  <arm_joint name="${l01}_to_${l02}" type="revolute"
-             axis_xyz="0 1 0"
-             limit_angle="1.57"
-             origin_rpy="0 0 0" origin_xyz="0 0 ${body_h}"
-             parent="${l01}"
+  <arm_joint_trans name="${l01}_to_${l02}" type="revolute"
+                   axis_xyz="0 1 0"
+                   limit="1.57"
+                   origin_rpy="0 0 0" origin_xyz="0 0 ${body_h}"
+                   parent="${l01}"
              child="${l02}"/>
   <arm_box name="${l02}"
@@ -57,17 +58,109 @@
            izz="1"
            size="${body_w} ${body_l} ${body_h}"/>
-  <arm_joint name="${l02}_to_${l0h}" type="revolute"
-             axis_xyz="0 1 0"
-             limit_angle="0.785"
-             origin_rpy="0 1.57 0" origin_xyz="0 0 ${body_h}"
-             parent="${l02}"
-             child="${l0h}"/>
+  <arm_joint_trans name="${l02}_to_${l0h}" type="revolute"
+                   axis_xyz="0 1 0"
+                   limit="0.785"
+                   origin_rpy="0 1.57 0" origin_xyz="0 0 ${body_h}"
+                   parent="${l02}"
+                   child="${l0h}"/>
   <arm_box name="${l0h}"
            mass="${head_mass}"
-           origin_rpy="0 0 0" origin_xyz="${head_x} 0 0"
+           origin_rpy="0 0 0" origin_xyz="${head_x} ${head_y} ${head_z}"
            ixx="1" ixy="0" ixz="0"
            iyy="1" iyz="0"
            izz="1"
            size="${head_w} ${head_l} ${head_h}"/>
+  <!-- End Effector - Telescopic Head -->
+  <arm_joint_dl_trans name="${l0h}_to_${m0d}" type="prismatic"
+                      axis_xyz="0 0 1"
+                      lower="0.00" upper="0.47"
+                      origin_rpy="0 0 0" origin_xyz="${drillm_x} ${drillm_y} ${drillm_z}"
+                      parent="${l0h}"
+                      child="${m0d}"/>
+  <arm_cylinder name="${m0d}"
+                mass="${drillm_mass}"
+                origin_rpy="0 0 0" origin_xyz="0 0 0"
+                ixx="1" ixy="0" ixz="0"
+                iyy="1" iyz="0"
+                izz="1"
+                radius="${drillm_r}" length="${drillm_l}"/>
+  <arm_joint_con_trans name="${m0d}_to_${edma}"
+                       axis_xyz="0 0 1"
+                       origin_rpy="0 0 0" origin_xyz="0 0 ${drillm_zz}"
+                       parent="${m0d}"
+                       child="${edma}"/>
+  <arm_cylinder name="${edma}"
+                mass="${drillma_mass}"
+                origin_rpy="0 0 0" origin_xyz="0 0 ${drillma_z}"
+                ixx="1" ixy="0" ixz="0"
+                iyy="1" iyz="0"
+                izz="1"
+                radius="${drillma_r}" length="${drillma_l}"/>
+  <!-- End Effector Alternative Head -->
+  <arm_joint_trans name="${l0h}_to_${e0t}" type="revolute"
+                   axis_xyz="0 0 1"
+                   limit="0.785"
+                   origin_rpy="0 0 0" origin_xyz="${TT_x} ${TT_y} ${TT_z}"
+                   parent="${l0h}"
+                   child="${e0t}"/>
+  <arm_cylinder name="${e0t}"
+                mass="${TT_mass}"
+                origin_rpy="0 0 0" origin_xyz="0 0 0"
+                ixx="1" ixy="0" ixz="0"
+                iyy="1" iyz="0"
+                izz="1"
+                radius="${TT_r}" length="${TT_l}"/>
+  <arm_joint_dl_trans name="${e0t}_to_${e0db}" type="prismatic"
+                      axis_xyz="0 0 1"
+                      lower="0.00" upper="0.43"
+                      origin_rpy="0 0 0" origin_xyz="${drillb_x} 0 ${tool_z}"
+                      parent="${e0t}"
+                      child="${e0db}"/>
+  <arm_cylinder name="${e0db}"
+                mass="${drillb_mass}"
+                origin_rpy="0 0 0" origin_xyz="0 0 ${drillb_z}"
+                ixx="1" ixy="0" ixz="0"
+                iyy="1" iyz="0"
+                izz="1"
+                radius="${drillb_r}" length="${drillb_l}"/>
+  <arm_joint_dl_trans name="${e0t}_to_${e0ds}" type="prismatic"
+                      axis_xyz="0 0 1"
+                      lower="0.00" upper="0.43"
+                      origin_rpy="0 0 0" origin_xyz="${drills_x} ${drills_y} ${tool_z}"
+                      parent="${e0t}"
+                      child="${e0ds}"/>
+  <arm_cylinder name="${e0ds}"
+                mass="${drills_mass}"
+                origin_rpy="0 0 0" origin_xyz="0 0 ${drills_z}"
+                ixx="1" ixy="0" ixz="0"
+                iyy="1" iyz="0"
+                izz="1"
+                radius="${drills_r}" length="${drills_l}"/>
+  <arm_joint_dl_trans name="${e0t}_to_${e0sd}" type="prismatic"
+                      axis_xyz="0 0 1"
+                      lower="0.00" upper="0.43"
+                      origin_rpy="0 0 0" origin_xyz="${SD_x} ${SD_y} ${tool_z}"
+                      parent="${e0t}"
+                      child="${e0sd}"/>
+  <arm_cylinder name="${e0sd}"
+                mass="${SD_mass}"
+                origin_rpy="0 0 0" origin_xyz="0 0 ${SD_z}"
+                ixx="1" ixy="0" ixz="0"
+                iyy="1" iyz="0"
+                izz="1"
+                radius="${SD_r}" length="${SD_l}"/>
+  <!-- End Effector - Ending Tube -->
+  <joint name="ending_tube_position_joint" type="fixed">
+    <origin rpy="0 0 0" xyz="${ET_x} ${ET_y} ${ET_z}"/>
+    <parent link="head_link"/>
+    <child link="e0e"/>
+  </joint>
+  <arm_cylinder name="e0e"
+                mass="${ET_mass}"
+                origin_rpy="0 0 0" origin_xyz="0 0 ${ET_zz}"
+                ixx="1" ixy="0" ixz="0"
+                iyy="1" iyz="0"
+                izz="1"
+                radius="${ET_r}" length="${ET_l}"/>
   <!-- END - Robot Description -->
   <gazebo>

File: catkin_ws/src/arm_description/urdf/links_joints.xacro (robot description, xacro)
@@ -3,12 +3,82 @@
 <!-- This document describes the global functions -->
 <!--      Machenical Practice Testing Version     -->
-<!--           Last editted: 11/01, 2018          -->
+<!--           Last editted: 11/18, 2018          -->
 <!--               Editor: Wolf Chen              -->
 <robot xmlns:xacro="http://www.ros.org/wiki/xacro">
   <!-- Define the "joint" description -->
-  <xacro:macro name="arm_joint" params="name type axis_xyz limit_angle origin_rpy origin_xyz parent child">
+  <xacro:macro name="arm_joint_s" params="name type axis_xyz limit origin_rpy origin_xyz parent child">
     <joint name="${name}" type="${type}">
       <axis xyz="${axis_xyz}"/>
-      <limit effort="1000.0" lower="-${limit_angle}" upper="${limit_angle}" velocity="0.2"/>
+      <limit effort="1000.0" lower="-${limit}" upper="${limit}" velocity="0.2"/>
+      <!-- Define the origin of the NEXT link -->
+      <origin rpy="${origin_rpy}" xyz="${origin_xyz}"/>
+      <parent link="${parent}"/>
+      <child link="${child}"/>
+    </joint>
+  </xacro:macro>
+  <xacro:macro name="arm_joint_dl_s" params="name type axis_xyz lower upper origin_rpy origin_xyz parent child">
+    <joint name="${name}" type="${type}">
+      <axis xyz="${axis_xyz}"/>
+      <limit effort="1000.0" lower="-${lower}" upper="${upper}" velocity="0.2"/>
+      <!-- Define the origin of the NEXT link -->
+      <origin rpy="${origin_rpy}" xyz="${origin_xyz}"/>
+      <parent link="${parent}"/>
+      <child link="${child}"/>
+    </joint>
+  </xacro:macro>
+  <xacro:macro name="arm_joint_con_s" params="name axis_xyz origin_rpy origin_xyz parent child">
+    <joint name="${name}" type="continuous">
+      <axis xyz="${axis_xyz}"/>
+      <limit effort="1000.0" velocity="0.2"/>
+      <!-- Define the origin of the NEXT link -->
+      <origin rpy="${origin_rpy}" xyz="${origin_xyz}"/>
+      <parent link="${parent}"/>
+      <child link="${child}"/>
+    </joint>
+  </xacro:macro>
+  <xacro:macro name="arm_joint" params="name type axis_xyz limit origin_rpy origin_xyz parent child">
+    <joint name="${name}" type="${type}">
+      <axis xyz="${axis_xyz}"/>
+      <limit effort="1000.0" lower="-${limit}" upper="${limit}" velocity="0.2"/>
+      <!-- Define the origin of the NEXT link -->
+      <origin rpy="${origin_rpy}" xyz="${origin_xyz}"/>
+      <parent link="${parent}"/>
+      <child link="${child}"/>
+    </joint>
+    <transmission name="trans_${name}">
+      <type>transmission_interface/SimpleTransmission</type>
+      <joint name="${name}">
+        <hardwareInterface>hardware_interface/EffortJointInterface</hardwareInterface>
+      </joint>
+      <actuator name="motor_${name}">
+        <hardwareInterface>hardware_interface/EffortJointInterface</hardwareInterface>
+        <mechanicalReduction>1</mechanicalReduction>
+      </actuator>
+    </transmission>
+  </xacro:macro>
+  <xacro:macro name="arm_joint_dl" params="name type axis_xyz lower upper origin_rpy origin_xyz parent child">
+    <joint name="${name}" type="${type}">
+      <axis xyz="${axis_xyz}"/>
+      <limit effort="1000.0" lower="-${lower}" upper="${upper}" velocity="0.2"/>
+      <!-- Define the origin of the NEXT link -->
+      <origin rpy="${origin_rpy}" xyz="${origin_xyz}"/>
+      <parent link="${parent}"/>
+      <child link="${child}"/>
+    </joint>
+    <transmission name="trans_${name}">
+      <type>transmission_interface/SimpleTransmission</type>
+      <joint name="${name}">
+        <hardwareInterface>hardware_interface/EffortJointInterface</hardwareInterface>
+      </joint>
+      <actuator name="motor_${name}">
+        <hardwareInterface>hardware_interface/EffortJointInterface</hardwareInterface>
+        <mechanicalReduction>1</mechanicalReduction>
+      </actuator>
+    </transmission>
+  </xacro:macro>
+  <xacro:macro name="arm_joint_con" params="name axis_xyz origin_rpy origin_xyz parent child">
+    <joint name="${name}" type="continuous">
+      <axis xyz="${axis_xyz}"/>
+      <limit effort="1000.0" velocity="0.2"/>
       <!-- Define the origin of the NEXT link -->
       <origin rpy="${origin_rpy}" xyz="${origin_xyz}"/>
@@ -28,5 +98,5 @@
   </xacro:macro>
   <!-- Define the "arm body" description -->
-  <xacro:macro name="arm_cylinder" params="name mass origin_rpy origin_xyz ixx ixy ixz iyy iyz izz radius length">
+  <xacro:macro name="arm_cylinder" params="name mass origin_rpy origin_xyz ixx ixy ixz iyy iyz izz radius length color_name color">
     <link name="${name}">
       <inertial>
@@ -45,9 +115,12 @@
         <geometry>
           <cylinder radius="${radius}" length="${length}"/>
+          <material name="${color_name}">
+            <color rgba="${color}"/>
+          </material>
         </geometry>
       </visual>
     </link>
   </xacro:macro>
-  <xacro:macro name="arm_box" params="name mass origin_rpy origin_xyz ixx ixy ixz iyy iyz izz size">
+  <xacro:macro name="arm_box" params="name mass origin_rpy origin_xyz ixx ixy ixz iyy iyz izz size color_name color">
     <link name="${name}">
       <inertial>
@@ -66,4 +139,7 @@
         <geometry>
           <box size="${size}"/>
+          <material name="${color_name}">
+            <color rgba="${color}"/>
+          </material>
         </geometry>
       </visual>
@@ -71,11 +147,11 @@
   </xacro:macro>
   <!-- Define the "transmission" description -->
-  <xacro:macro name="arm_transmission" params="name joint_name motor_name">
-    <transmission name="${name}">
+  <xacro:macro name="arm_trans" params="name">
+    <transmission name="trans_${name}">
       <type>transmission_interface/SimpleTransmission</type>
-      <joint name="${joint_name}">
+      <joint name="${name}">
         <hardwareInterface>hardware_interface/EffortJointInterface</hardwareInterface>
       </joint>
-      <actuator name="${motor_name}">
+      <actuator name="motor_${name}">
         <hardwareInterface>hardware_interface/EffortJointInterface</hardwareInterface>
         <mechanicalReduction>1</mechanicalReduction>

File: catkin_ws/src/arm_description/urdf/robot_parameters.xacro (robot description, xacro)
@@ -3,5 +3,5 @@
 <!-- This document describes the names and parameters -->
 <!--        Machenical Practice Testing Version       -->
-<!--             Last editted: 11/01, 2018            -->
+<!--             Last editted: 11/17, 2018            -->
 <!--                 Editor: Wolf Chen                -->
 <robot xmlns:xacro="http://www.ros.org/wiki/xacro">
@@ -12,9 +12,19 @@
   <xacro:property name="l0h" value="head_link"/>
   <xacro:property name="m0b" value="base_motor"/>
+  <xacro:property name="m0d" value="drill_motor"/>
+  <xacro:property name="e0s" value="EE_screw"/>
+  <xacro:property name="e0L" value="EE_L-plate"/>
+  <xacro:property name="edma" value="EE_drill_motor_axis"/>
+  <xacro:property name="e0t" value="EE_turntable"/>
+  <xacro:property name="e0db" value="EE_drill_big"/>
+  <xacro:property name="e0ds" value="EE_drill_small"/>
+  <xacro:property name="e0sd" value="EE_screwdriver"/>
+  <xacro:property name="e0e" value="EE_ending_tube"/>
   <!-- True Names of Motors Description -->
   <xacro:property name="ground_motor_name" value="MG996R"/>
   <xacro:property name="base_motor_name" value="ARS-3216HTG+HV"/>
   <xacro:property name="body_motor_name" value="QDS-15RO"/>
-  <!-- Appearances Description -->
+  <xacro:property name="drill_motor_name" value="2212-1400KV"/>
+  <!-- Body Appearances Description -->
   <xacro:property name="base_r" value="0.65"/>
   <xacro:property name="base_l" value="0.75"/>
@@ -22,16 +32,60 @@
   <xacro:property name="body_l" value="0.50"/>
   <xacro:property name="body_h" value="2.15"/>
-  <xacro:property name="head_w" value="1.30"/>
-  <xacro:property name="head_l" value="1.20"/>
-  <xacro:property name="head_h" value="2.40"/>
+  <xacro:property name="head_w" value="1.20"/>
+  <xacro:property name="head_l" value="1.36"/>
+  <xacro:property name="head_h" value="2.8"/>
+  <!-- End Effector Appearances Description -->
+  <xacro:property name="screw_r" value="0.05"/>
+  <xacro:property name="screw_l" value="1.2"/>
+  <xacro:property name="L_w" value="0.6"/>
+  <xacro:property name="L_l" value="0.55"/>
+  <xacro:property name="L_h" value="0.08"/>
+  <xacro:property name="drillma_r" value="0.04"/>
+  <xacro:property name="drillma_l" value="0.66"/>
+  <xacro:property name="TT_r" value="0.4"/>
+  <xacro:property name="TT_l" value="0.2"/>
+  <xacro:property name="drillb_r" value="0.05"/>
+  <xacro:property name="drillb_l" value="0.89"/>
+  <xacro:property name="drills_r" value="0.05"/>
+  <xacro:property name="drills_l" value="0.82"/>
+  <xacro:property name="SD_r" value="0.05"/>
+  <xacro:property name="SD_l" value="0.87"/>
+  <xacro:property name="ET_r" value="0.0504"/>
+  <xacro:property name="ET_l" value="0.075"/>
   <!-- Motors Description -->
   <xacro:property name="basem_w" value="0.35"/>
   <xacro:property name="basem_l" value="0.40"/>
   <xacro:property name="basem_h" value="0.38"/>
-  <!-- Shape Origins Description -->
+  <xacro:property name="drillm_r" value="0.14"/>
+  <xacro:property name="drillm_l" value="0.29"/>
+  <!-- Body Shape Origins Description -->
   <xacro:property name="base_z" value="0.375"/>
   <xacro:property name="basem_z" value="0.19"/>
   <xacro:property name="body_z" value="1.075"/>
-  <xacro:property name="head_x" value="-0.65"/>
+  <xacro:property name="head_x" value="-0.60"/>
+  <xacro:property name="head_y" value="0.00"/>
+  <xacro:property name="head_z" value="0.40"/>
+  <!-- End Effector Origins Description -->
+  <xacro:property name="drillm_x" value="-0.7"/>
+  <xacro:property name="drillm_y" value="-0.06"/>
+  <xacro:property name="drillm_z" value="-0.135"/>
+  <xacro:property name="drillm_zz" value="0.145"/>
+  <xacro:property name="drillma_z" value="0.34"/>
+  <xacro:property name="TT_x" value="-0.394"/>
+  <xacro:property name="TT_y" value="-0.06"/>
+  <xacro:property name="TT_z" value="0.78"/>
+  <xacro:property name="drillb_x" value="-0.306"/>
+  <xacro:property name="drillb_z" value="0.445"/>
+  <xacro:property name="drills_x" value="-0.216"/>
+  <xacro:property name="drills_y" value="0.216"/>
+  <xacro:property name="drills_z" value="0.41"/>
+  <xacro:property name="SD_x" value="-0.216"/>
+  <xacro:property name="SD_y" value="-0.216"/>
+  <xacro:property name="SD_z" value="0.435"/>
+  <xacro:property name="tool_z" value="-0.06"/>
+  <xacro:property name="ET_x" value="-0.7"/>
+  <xacro:property name="ET_y" value="-0.06"/>
+  <xacro:property name="ET_z" value="1.8"/>
+  <xacro:property name="ET_zz" value="0.0375"/>
   <!-- Physical Values Description -->
   <xacro:property name="base_mass" value="999"/>
@@ -39,3 +93,14 @@
   <xacro:property name="body_mass" value="2"/>
   <xacro:property name="head_mass" value="5"/>
+  <xacro:property name="drillm_mass" value="1"/>
+  <xacro:property name="drillma_mass" value="0.5"/>
+  <xacro:property name="TT_mass" value="0.25"/>
+  <xacro:property name="drillb_mass" value="0.25"/>
+  <xacro:property name="drills_mass" value="0.25"/>
+  <xacro:property name="SD_mass" value="0.25"/>
+  <xacro:property name="ET_mass" value="0.01"/>
+  <!-- Color Description -->
+  <xacro:property name="LGrey" value="0.7 0.7 0.7 1.0"/>
+  <xacro:property name="LGrey_T" value="0.7 0.7 0.7 0.5"/>
+  <xacro:property name="Black" value="1 1 1 1"/>
 </robot>
