Commit message: add arm3

File: catkin_ws/src/arm_description/urdf/robot_parameters.xacro (robot description, xacro)
@@ -34,5 +34,5 @@
   <xacro:property name="head_w" value="1.20"/>
   <xacro:property name="head_l" value="1.36"/>
-  <xacro:property name="head_h" value="2.8"/>
+  <xacro:property name="head_h" value="2.80"/>
   <!-- End Effector Appearances Description -->
   <xacro:property name="screw_r" value="0.05"/>

File: catkin_ws/src/arm_description/urdf/robot_parameters_ext.xacro (robot description, xacro)
@@ -9,4 +9,6 @@
   <xacro:property name="l0h2" value="head_link_2"/>
   <xacro:property name="sd02" value="small_drill_2"/>
+  <xacro:property name="l012" value="link_01_2"/>
+  <xacro:property name="l022" value="link_02_2"/>
   <!-- Body Appearance Description -->
   <xacro:property name="head_w_2" value="0.86"/>
@@ -15,4 +17,5 @@
   <xacro:property name="drills_r" value="0.02"/>
   <xacro:property name="drills_l" value="1.28"/>
+  <xacro:property name="body_h_2" value="1.05"/>
   <!-- Mass Description -->
   <xacro:property name="head_mass_2" value="2"/>
@@ -23,3 +26,4 @@
   <xacro:property name="drills_y_2" value="0"/>
   <xacro:property name="drills_z_2" value="0.165"/>
+  <xacro:property name="body_z_2" value="0.525"/>
 </robot>
