Commit message: arm3

File: catkin_ws/src/arm_description/urdf/arm3.urdf.xacro (robot description, xacro)
@@ -40,32 +40,32 @@
              origin_rpy="0 0 0" origin_xyz="0 0 ${basem_h}"
              parent="${m0b}"
-             child="${l012}"/>
-  <arm_box name="${l012}"
+             child="${l013}"/>
+  <arm_box name="${l013}"
            mass="${body_mass}"
-           origin_rpy="0 0 0" origin_xyz="0 0 ${body_z_2}"
+           origin_rpy="0 0 0" origin_xyz="0 0 ${body_z_3}"
            ixx="1" ixy="0" ixz="0"
            iyy="1" iyz="0"
            izz="1"
-           size="${body_w} ${body_l} ${body_h_2}"
+           size="${body_w} ${body_l} ${body_h_3}"
            color_name="LightGrey" color="${LGrey}"/>
   <arm_joint name="elbow_joint" type="revolute"
              axis_xyz="0 1 0"
              limit="1.57"
-             origin_rpy="0 0 0" origin_xyz="0 0 ${body_h_2}"
-             parent="${l012}"
-             child="${l022}"/>
-  <arm_box name="${l022}"
+             origin_rpy="0 0 0" origin_xyz="0 0 ${body_h_3}"
+             parent="${l013}"
+             child="${l023}"/>
+  <arm_box name="${l023}"
            mass="${body_mass}"
-           origin_rpy="0 0 0" origin_xyz="0 0 ${body_z_2}"
+           origin_rpy="0 0 0" origin_xyz="0 0 ${body_z_3}"
            ixx="1" ixy="0" ixz="0"
            iyy="1" iyz="0"
            izz="1"
-           size="${body_w} ${body_l} ${body_h_2}"
+           size="${body_w} ${body_l} ${body_h_3}"
            color_name="LightGrey" color="${LGrey}"/>
   <arm_joint name="wrist_joint" type="revolute"
              axis_xyz="0 1 0"
              limit="0.785"
-             origin_rpy="0 1.57 0" origin_xyz="0 0 ${body_h_2}"
-             parent="${l022}"
+             origin_rpy="0 1.57 0" origin_xyz="0 0 ${body_h_3}"
+             parent="${l023}"
              child="${l0h2}"/>
   <arm_box name="${l0h2}"

File: catkin_ws/src/arm_description/urdf/robot_parameters_ext.xacro (robot description, xacro)
@@ -6,4 +6,5 @@
 <!--                 Editor: Wolf Chen                -->
 <robot xmlns:xacro="http://www.ros.org/wiki/xacro">
+  <!-- Arm2 -->
   <!-- Name Description -->
   <xacro:property name="l0h2" value="head_link_2"/>
@@ -27,3 +28,11 @@
   <xacro:property name="drills_z_2" value="0.165"/>
   <xacro:property name="body_z_2" value="0.525"/>
+  <!-- Arm3 -->
+  <!-- Name Description -->
+  <xacro:property name="l013" value="link_01_3"/>
+  <xacro:property name="l023" value="link_02_3"/>
+  <!-- Body Appearance Description -->
+  <xacro:property name="body_h_3" value="1.15"/>
+  <!-- Origin Description -->
+  <xacro:property name="body_z_3" value="0.575"/>
 </robot>
